Commit message: changed macro name to robot_cell

File: urdf/robot_cell.urdf.xacro (robot description, xacro)
@@ -2,5 +2,5 @@
 <robot name="robot_cell" xmlns:xacro="https://ros.org/wiki/xacro">
     <xacro:include filename="$(find robot_cell_description)/urdf/robot_cell_macro.xacro"/>
-    <xacro:arg name="ur_type" default="ur10"/>
+    <xacro:arg name="ur_type" default="ur10e"/>
     <xacro:arg name="joint_limits_parameters_file" default="$(find ur_description)/config/$(arg ur_type)/joint_limits.yaml"/>
     <xacro:arg name="kinematics_parameters_file" default="$(find ur_description)/config/$(arg ur_type)/default_kinematics.yaml"/>
@@ -9,5 +9,5 @@
     <link name="world"/>
     <!-- This will create the scene where the robot is located in -->
-    <xacro:assembled_robot
+    <xacro:robot_cell
         parent="world"
         ur_type="$(arg ur_type)"
@@ -18,4 +18,4 @@
         >
             <origin xyz="0 0 0" rpy="0 0 0"/>
-    </xacro:assembled_robot>
+    </xacro:robot_cell>
 </robot>

File: urdf/robot_cell_macro.xacro (robot description, xacro)
@@ -11,5 +11,5 @@
     </material>
     <xacro:property name="gripper_name" value="robotiq_85"/>
-    <xacro:macro name="assembled_robot" params="
+    <xacro:macro name="robot_cell" params="
         parent
         *origin
