Commit message: changed the position of the robot with respect to word

File: urdf/robot_cell_macro.xacro (robot description, xacro)
@@ -30,5 +30,5 @@
             visual_parameters_file="${visual_parameters_file}"
         >
-            <origin xyz="0 0 ${height}" rpy="0 0 ${pi}"/>
+            <origin xyz="0 0 0" rpy="0 0 0"/>
         </xacro:ur_robot>
         <!-- This will create gripper -->

Commit message: robot_mount added. This fixes some issue with TF

File: urdf/robot_cell_macro.xacro (robot description, xacro)
@@ -20,13 +20,20 @@
         visual_parameters_file
         ">
+        <link name="robot_mount"/>
+        <joint name="base_to_robot_mount" type="fixed">
+            <parent link="${parent}"/>
+            <child link="robot_mount"/>
+            <origin xyz=" 0 0 0" rpy="0 0 0"/>
+        </joint>
         <!-- This will create the specific robot -->
         <xacro:ur_robot
             name="${ur_type}"
             tf_prefix="${ur_type}_"
-            parent="${parent}"
+            parent="robot_mount"
             joint_limits_parameters_file="${joint_limits_parameters_file}"
             kinematics_parameters_file="${kinematics_parameters_file}"
             physical_parameters_file="${physical_parameters_file}"
             visual_parameters_file="${visual_parameters_file}"
+            generate_ros2_control_tag="false"
         >
             <origin xyz="0 0 0" rpy="0 0 0"/>

Commit message: gripper_base link and joint added

File: urdf/robot_cell_macro.xacro (robot description, xacro)
@@ -39,11 +39,17 @@
             <origin xyz="0 0 0" rpy="0 0 0"/>
         </xacro:ur_robot>
+        <link name="gripper_base"/>
+        <joint name="flange_to_gripper" type="fixed">
+            <parent link="${ur_type}_tool0"/>
+            <child link="gripper_base"/>
+            <origin xyz=" 0 0 0" rpy="0 0 0"/>
+        </joint>
         <!-- This will create gripper -->
         <xacro:robotiq_gripper
             name="RobotiqGripper"
             prefix="${ur_type}_"
-            parent="${ur_type}_flange"
+            parent="gripper_base"
         >
-            <origin xyz="0 0 0" rpy="0 ${pi/2} 0"/>
+            <origin xyz="0 0 0" rpy="0 0 ${pi}"/>
         </xacro:robotiq_gripper>
         <!-- This will create tool -->
