Commit message: adjusted tool orientation

File: urdf/tool_macro.xacro (robot description, xacro)
@@ -22,5 +22,5 @@
                         Therefore, scaling down the pointer.
                     -->
-                    <mesh filename="package://robot_cell_description/meshes/pointer_v3.STL" scale="0.001 0.001 0.001"/>
+                    <mesh filename="package://robot_cell_description/meshes/pointer_v3-1.stl" scale="0.001 0.001 0.001"/>
                 </geometry>
                 <material name="red"/>
@@ -29,5 +29,5 @@
             <collision>
                 <geometry>
-                    <mesh filename="package://robot_cell_description/meshes/pointer_v3.STL" scale="0.001 0.001 0.001"/>
+                    <mesh filename="package://robot_cell_description/meshes/pointer_v3-1.stl" scale="0.001 0.001 0.001"/>
                 </geometry>
                 <origin xyz="0 0 0"/>
@@ -38,5 +38,5 @@
             <parent link="${parent}"/>
             <child link="${prefix}${name}"/>
-            <origin xyz="0 0 0.187" rpy="-${pi/2} 0 0"/>
+            <origin xyz="0 0 0.093" rpy="0 ${-pi/2} ${pi/2}"/>
         </joint>
     </xacro:macro>

Commit message: tip link and joint added to the tool

File: urdf/tool_macro.xacro (robot description, xacro)
@@ -40,4 +40,10 @@
             <origin xyz="0 0 0.093" rpy="0 ${-pi/2} ${pi/2}"/>
         </joint>
+        <link name="${prefix}tip" />
+        <joint name="${prefix}${name}_to_tip" type="fixed">
+            <parent link="${prefix}${name}"/>
+            <child link="${prefix}tip"/>
+            <origin xyz="0.22 0 0.011" rpy="0 0.982 0"/>
+        </joint>
     </xacro:macro>
 </robot>

Commit message: tip frame position added as per CAD design specs

File: urdf/tool_macro.xacro (robot description, xacro)
@@ -44,5 +44,5 @@
             <parent link="${prefix}${name}"/>
             <child link="${prefix}tip"/>
-            <origin xyz="0.22 0 0.011" rpy="0 0.982 0"/>
+            <origin xyz="0.211 0 0" rpy="0 ${pi/3} 0"/>
         </joint>
     </xacro:macro>

Commit message: tool tip frame position updated

File: urdf/tool_macro.xacro (robot description, xacro)
@@ -38,5 +38,5 @@
             <parent link="${parent}"/>
             <child link="${prefix}${name}"/>
-            <origin xyz="0 0 0.093" rpy="0 ${-pi/2} ${pi/2}"/>
+            <origin xyz="0 0 0.11505" rpy="0 ${-pi/2} ${pi/2}"/>
         </joint>
         <link name="${prefix}tip" />
